Commit message: ft sensor can work in gazebo

File: robotiq_ft_sensor_description/urdf/examples_of_macros/example_use_robotiq_ft300.xacro (robot description, xacro)
@@ -5,5 +5,5 @@
 <robot name="robotiq_arg2f_80_model" xmlns:xacro="http://ros.org/wiki/xacro">
   <!--Import macro for left arm gripper-->
-  <xacro:include filename="$(find robotiq_ft_sensor)/urdf/robotiq_ft300.urdf.xacro" />
+  <xacro:include filename="$(find robotiq_ft_sensor_description)/urdf/robotiq_ft300.urdf.xacro" />
   <!--Base frame for reference-->
   <link name="world" />

File: robotiq_ft_sensor_description/urdf/robotiq_ft300.urdf.xacro (robot description, xacro)
@@ -6,5 +6,5 @@
         ```
             // Import this macro function
-            <xacro:include filename="$(find find robotiq_ft_sensor)/urdf/robotiq_ft300.urdf.xacro" />
+            <xacro:include filename="$(find find robotiq_ft_sensor_description)/urdf/robotiq_ft300.urdf.xacro" />
             // Instanciate sensor instance and connect it to robot flange
             <xacro:robotiq_ft300 parent="robot_flange_link" prefix="">
@@ -30,5 +30,5 @@
                 <origin xyz="0 0 0" rpy="0 0 0" />
                 <geometry>
-                    <mesh filename="file://$(find robotiq_ft_sensor)/meshes/visual/robotiq_ft300.STL"/>
+                    <mesh filename="file://$(find robotiq_ft_sensor_description)/meshes/visual/robotiq_ft300.STL"/>
                 </geometry>
                 <material name="Robotiq-Black">
@@ -39,5 +39,5 @@
                 <origin xyz="0 0 0" rpy="0 0 0" />
                 <geometry>
-                    <mesh filename="file://$(find robotiq_ft_sensor)/meshes/collision/robotiq_ft300.STL"/>
+                    <mesh filename="file://$(find robotiq_ft_sensor_description)/meshes/collision/robotiq_ft300.STL"/>
                 </geometry>
             </collision>
@@ -48,5 +48,5 @@
                 <origin xyz="0 0 0" rpy="0 0 0" />
                 <geometry>
-                    <mesh filename="file://$(find robotiq_ft_sensor)/meshes/visual/mountings/robotiq_ft300-G-062-COUPLING_G-50-4M6-1D6_20181119.STL"/>
+                    <mesh filename="file://$(find robotiq_ft_sensor_description)/meshes/visual/mountings/robotiq_ft300-G-062-COUPLING_G-50-4M6-1D6_20181119.STL"/>
                 </geometry>
                 <material name="Robotiq-Grey">
@@ -57,5 +57,5 @@
                 <origin xyz="0 0 0" rpy="0 0 0" />
                 <geometry>
-                    <mesh filename="file://$(find robotiq_ft_sensor)/meshes/collision/mountings/robotiq_ft300-G-062-COUPLING_G-50-4M6-1D6_20181119.STL"/>
+                    <mesh filename="file://$(find robotiq_ft_sensor_description)/meshes/collision/mountings/robotiq_ft300-G-062-COUPLING_G-50-4M6-1D6_20181119.STL"/>
                 </geometry>
             </collision>

File: robotiq_ft_sensor_description/urdf/robotiq_fts150.urdf.xacro (robot description, xacro)
@@ -18,5 +18,5 @@
                 <origin xyz="0 0 0" rpy="0 0 0" />
                 <geometry>
-                    <mesh filename="file://$(find robotiq_ft_sensor)/meshes/visual/robotiq_fts150.stl"/>
+                    <mesh filename="file://$(find robotiq_ft_sensor_description)/meshes/visual/robotiq_fts150.stl"/>
                 </geometry>
                 <material name="black"/>
@@ -25,5 +25,5 @@
                 <origin xyz="0 0 0" rpy="0 0 0" />
                 <geometry>
-                    <mesh filename="file://$(find robotiq_ft_sensor)/meshes/collision/robotiq_fts150.stl"/>
+                    <mesh filename="file://$(find robotiq_ft_sensor_description)/meshes/collision/robotiq_fts150.stl"/>
                 </geometry>
             </collision>

File: robotiq_ft_sensor_description/urdf/test.urdf (robot description, URDF)
Before this commit: robot test_ft_sensor_gazebo, 5 links, 4 joints
Links:
- removed link link1
- added link tip_link, mass 1.0; collision cylinder length=0.06 radius=0.015; visual cylinder length=0.06 radius=0.015
- link ft300_mounting_plate: geometry collision mesh filename=file:///home/xiaobaige/ur_project_ros2/install/robotiq_ft_s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; visual mesh filename=file:///home/xiaobaige/ur_project_ros2/install/robotiq_ft_s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
- link ft300_sensor: geometry collision mesh filename=file:///home/xiaobaige/ur_project_ros2/install/robotiq_ft_s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; visual mesh filename=file:///home/xiaobaige/ur_project_ros2/install/robotiq_ft_s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
Joints:
- joint ft300_fix: origin xyz=0 0 0.3 rpy=0 0 0 -> xyz=0 0 0.3 rpy=1.5707 0 0
- joint ft300_sensor_joint: child link1 -> tip_link; limit lower=0 upper=0 effort=1000 velocity=6.5 -> (none); type revolute -> fixed
